File: gateron_lp_kbd/gateron_lp_kbd.kicad_pcb (KiCad board)
At the start: 2 copper layers, 234.5 x 116.5 mm, 152 parts, among them J1 TYPE-C-31-M-12, J2 Battery JST-SH, Q1 DMG3415U, SW1 KS-33, SW10 KS-33, SW11 KS-33, SW12 KS-33, SW13 KS-33, SW14 KS-33, SW15 KS-33, SW16 KS-33, SW17 KS-33, SW18 KS-33, SW19 KS-33, SW2 KS-33, SW20 KS-33, SW21 KS-33, SW22 KS-33, SW23 KS-33, SW24 KS-33, SW25 KS-33, SW26 KS-33, SW27 KS-33, SW28 KS-33, SW29 KS-33, SW3 KS-33, SW30 KS-33, SW31 KS-33, SW32 KS-33, SW33 KS-33, SW34 KS-33, SW35 KS-33, SW36 KS-33, SW37 KS-33, SW38 KS-33, SW39 KS-33, SW4 KS-33, SW40 KS-33, SW41 KS-33, SW42 KS-33, SW43 KS-33, SW44 KS-33, SW45 KS-33, SW46 KS-33, SW47 KS-33, SW48 KS-33, SW49 KS-33, SW5 KS-33, SW50 KS-33, SW51 KS-33, SW52 KS-33, SW53 KS-33, SW54 KS-33, SW55 KS-33, SW56 KS-33, SW57 KS-33, SW58 KS-33, SW59 KS-33, SW6 KS-33, SW60 RESET, SW61 BOOT, SW62 PWR MSK-12C02, SW7 KS-33, SW8 KS-33, SW9 KS-33, U1 ESP32-C6-MINI-1, U2 MCP73831, U3 AP2112K-3.3, U4 USBLC6-2SC6

Commit message: Add RP2040 board routing engine, reverse-mount LED redesign, and 3D models
- New route_kbd_rp2040.py: deterministic + A*-hybrid autorouter for the
  RP2040 variant. Hand-routes the congested ROW/COL matrix fanout and
  QSPI north strip net-by-net (verified against the real clearance
  checker), falls back to generic A* elsewhere, and heals remaining
  gaps in a final pass.
- Redesigned the per-key RGB LED footprint (fp_sk6812mini) to a real
  reverse-mount part on B.Cu with a light-transmission cutout, matching
  a verified KiCad reference footprint instead of a hand-derived one.
- Added 3D models to ~15 footprints across both board variants (via
  add_3d.py for the ESP32 variant, inline `model()` blocks for RP2040)
  and synced datasheets for real part verification.
- Fixed several real bugs surfaced while routing: VSYS's per-LED
  routing referenced the wrong pin after the LED footprint redesign
  (silently trying to via into GND on all 59 LEDs); the matching
  per-LED decoupling caps sat in the ~0mm gap between the LED's own
  cutout and the next row's switch leg hole; C33 was placed closer to
  BOOTSEL's through-hole pad than any trace could legally clear;
  BOOTSEL's own switch had two same-named leg pads that were never
  wired together; VBAT_SENSE's escape route was getting walled off by
  whichever of XIN/XOUT happened to route first.
- Board currently routes cleanly except for a known cluster of nets
  (+3V3, DVDD, QSPI_SCLK/SD2/SD3, RGB_GPIO, USB_DM/DP, VREG_VIN) all
  bottlenecked by the same over-saturated escape corridor next to U1 --
  next up for a dedicated deterministic-routing pass.

Co-Authored-By: Claude Sonnet 5 <noreply@anthropic.com>
Routing:
- net GND: track 49.0 -> 43.4 mm, vias 36 -> 33
- net USB_DM: track 126.5 -> 124.7 mm
- net BAT+: track 110.2 -> 108.4 mm
- net VBUS: track 162.7 -> 163.9 mm
- net USB_DP: track 122.3 -> 123.1 mm
Other:
- board text added: "Gateron LP 5x12 - ESP32-C6 wireless"
- board text removed: "SMK LP 5x12 - ESP32-C6 wireless"
