File: gateron_lp_kbd_rp2040/gateron_lp_kbd_rp2040.kicad_sch (KiCad schematic)
At the start: 300 parts, among them J1 TYPE-C-31-M-12, J2 JST-SH-2 SM02B, Q1 DMG3415U, SW1 KS-33, SW10 KS-33, SW11 KS-33, SW12 KS-33, SW13 KS-33, SW14 KS-33, SW15 KS-33, SW16 KS-33, SW17 KS-33, SW18 KS-33, SW19 KS-33, SW2 KS-33, SW20 KS-33, SW21 KS-33, SW22 KS-33, SW23 KS-33, SW24 KS-33, SW25 KS-33, SW26 KS-33, SW27 KS-33, SW28 KS-33, SW29 KS-33, SW3 KS-33, SW30 KS-33, SW31 KS-33, SW32 KS-33, SW33 KS-33, SW34 KS-33, SW35 KS-33, SW36 KS-33, SW37 KS-33, SW38 KS-33, SW39 KS-33, SW4 KS-33, SW40 KS-33, SW41 KS-33, SW42 KS-33, SW43 KS-33, SW44 KS-33, SW45 KS-33, SW46 KS-33, SW47 KS-33, SW48 KS-33, SW49 KS-33, SW5 KS-33, SW50 KS-33, SW51 KS-33, SW52 KS-33, SW53 KS-33, SW54 2U, SW55 KS-33, SW56 KS-33, SW57 KS-33, SW58 KS-33, SW59 KS-33, SW6 KS-33, SW60 RESET, SW61 BOOTSEL (VERIFY), SW62 PWR MSK-12C02, SW7 KS-33, SW8 KS-33, SW9 KS-33, U1 RP2040, U2 MCP73831-2ACI/OT, U3 AP2112K-3.3, U4 USBLC6-2SC6, U5 W25Q16JVUXIQ, U6 CYW43439, U7 SN74AHCT1G125DBVR, Y1 12MHz, Y2 37.4MHz

Commit message: Relocate U5 flash beside the QSPI bank; route all 7 stuck nets + RF feed
The QSPI flash sat SOUTH-EAST of U1 while the QSPI pins exit NORTH, so
every QSPI line wrapped around U1's east side. The lane/elevator system
that required (QSPI_SD1's F lane at y=23.75 spanning x 152.55-170, plus
the x=170-174 elevators) sealed the whole U1-north pocket -- QSPI_SD2/
SCLK/SD3, XIN, VREG_VIN and USB_DM/DP were all unroutable behind it,
which is what the last ~10 commits kept hitting from different angles.

U5 now sits at (149.8, 24.0), directly west of the QSPI pin bank (the
Pico reference design's arrangement), with C15 (its VCC cap, now 0402)
alongside. QSPI escape stubs get hand-picked depths instead of the
uniform staircase: SD3/SCLK/SD0's tips land exactly on U5's east-column
pad rows (three dead-straight lanes), SS/SD1/SD2 wrap U5's south-west
corner into the west column -- all emitted as must_clear_seg-verified
deterministic copper. The old lane/elevator code and the forced skips
for QSPI_SD2/SCLK/SD3 are deleted.

Knock-on fixes, each found by the emit-time clearance assertions:
- claim-order restructure: USB_DM's jogs, then v43/v48/v49 (2mm search
  radius, most fragile), then the DVDD pin-45/50 via gather, then
  VREG_VIN's jog -- all before the minimum-system A* nets are free to
  claim the reopened pocket's corridors
- XIN routes before XOUT (and C13-first): XIN's escape tip sits one
  pin-pitch inside XOUT's, so whichever routes first claims the only
  southern corridor; XOUT's east-pad target is the easier second
- +3V3 pin 33's In1 expressway retargeted to C11's pad (its old landing
  spot was C15's now-vacated position), passing south of DVDD's riser
- QSPI_SS's redundant second chain removed (the SW wrap already ties
  U5.1 to the stub)
- WLRF_ANT_MID feed is deterministic 0.4mm RF copper: generic A* can
  never route it (the mask bans the whole antenna keepout, and a 0.4mm
  trace can only attach to L2's 0201 pad at its outer edge). Riser at
  x=47.5 between U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
Parts:
- C15: footprint kbd:RC_0603 -> kbd:RC_0402
Changed lines of the file:
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@@
     (property "Reference" "C15" (at 96.52 109.22 0) (effects (font (size 1.27 1.27))))
     (property "Value" "100n" (at 96.52 119.38 0) (effects (font (size 1.27 1.27))))
-    (property "Footprint" "kbd:RC_0603" (at 96.52 114.3 0) (effects (font (size 1.27 1.27)) (hide yes)))
+    (property "Footprint" "kbd:RC_0402" (at 96.52 114.3 0) (effects (font (size 1.27 1.27)) (hide yes)))
     (property "Datasheet" "~" (at 96.52 114.3 0) (effects (font (size 1.27 1.27)) (hide yes)))
     (property "Description" "" (at 96.52 114.3 0) (effects (font (size 1.27 1.27)) (hide yes)))

Commit message: BOM: key positions are the hot-swap socket, not the switch
The soldered part at each key position is the Gateron KS-2P02B01-02
hot-swap socket -- the KS-33 switch (and keycap) plug in and are
user-installed, ordered from keyboard vendors rather than with the PCB
parts. The BOM previously listed 59x "KS-33" (58 + one "2U") and no
socket at all, so nothing reminded anyone to order the one part that
actually gets reflowed.

- sym_inst() grows a props= param for extra hidden symbol properties
- SW1-59 now carry Value/MPN "KS-2P02B01-02", Manufacturer "Gateron",
  and a BOM Comment noting the switch/keycap are separate purchases
  (plus a 2U keycap/stabilizer note on SW54)
- footprint Value matches, keeping sch/PCB cross-checks clean
- BOM collapses to one clean 59x socket line (43 lines total)

Note: the footprint still has exclude_from_pos_files (inherited from
when it modeled the switch) -- if the sockets are ever machine-placed
by an assembly service, that flag needs to go.

Co-Authored-By: Claude Fable 5 <noreply@anthropic.com>
Parts:
- SW1, SW10, SW11, SW12, SW13, SW14, SW15, SW16, SW17, SW18, SW19, SW2, SW20, SW21, SW22, SW23, SW24, SW25, SW26, SW27, SW28, SW29, SW3, SW30, SW31, SW32, SW33, SW34, SW35, SW36, SW37, SW38, SW39, SW4, SW40, SW41, SW42, SW43, SW44, SW45, SW46, SW47, SW48, SW49, SW5, SW50, SW51, SW52, SW53, SW55, SW56, SW57, SW58, SW59, SW6, SW7, SW8, SW9: value KS-33 -> KS-2P02B01-02; BOM Comments (none) -> Hot-swap socket (soldered, PCB assembly). The Gateron KS-33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; MPN (none) -> KS-2P02B01-02; Manufacturer (none) -> Gateron
- SW54: value 2U -> KS-2P02B01-02; BOM Comments (none) -> Hot-swap socket (soldered, PCB assembly). The Gateron KS-33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; MPN (none) -> KS-2P02B01-02; Manufacturer (none) -> Gateron
