File: gateron_lp_kbd_rp2040/gateron_lp_kbd_rp2040.kicad_sch (KiCad schematic)
At the start: 300 parts, among them J1 TYPE-C-31-M-12, J2 JST-SH-2 SM02B, Q1 DMG3415U, SW1 KS-2P02B01-02, SW10 KS-2P02B01-02, SW11 KS-2P02B01-02, SW12 KS-2P02B01-02, SW13 KS-2P02B01-02, SW14 KS-2P02B01-02, SW15 KS-2P02B01-02, SW16 KS-2P02B01-02, SW17 KS-2P02B01-02, SW18 KS-2P02B01-02, SW19 KS-2P02B01-02, SW2 KS-2P02B01-02, SW20 KS-2P02B01-02, SW21 KS-2P02B01-02, SW22 KS-2P02B01-02, SW23 KS-2P02B01-02, SW24 KS-2P02B01-02, SW25 KS-2P02B01-02, SW26 KS-2P02B01-02, SW27 KS-2P02B01-02, SW28 KS-2P02B01-02, SW29 KS-2P02B01-02, SW3 KS-2P02B01-02, SW30 KS-2P02B01-02, SW31 KS-2P02B01-02, SW32 KS-2P02B01-02, SW33 KS-2P02B01-02, SW34 KS-2P02B01-02, SW35 KS-2P02B01-02, SW36 KS-2P02B01-02, SW37 KS-2P02B01-02, SW38 KS-2P02B01-02, SW39 KS-2P02B01-02, SW4 KS-2P02B01-02, SW40 KS-2P02B01-02, SW41 KS-2P02B01-02, SW42 KS-2P02B01-02, SW43 KS-2P02B01-02, SW44 KS-2P02B01-02, SW45 KS-2P02B01-02, SW46 KS-2P02B01-02, SW47 KS-2P02B01-02, SW48 KS-2P02B01-02, SW49 KS-2P02B01-02, SW5 KS-2P02B01-02, SW50 KS-2P02B01-02, SW51 KS-2P02B01-02, SW52 KS-2P02B01-02, SW53 KS-2P02B01-02, SW54 KS-2P02B01-02, SW55 KS-2P02B01-02, SW56 KS-2P02B01-02, SW57 KS-2P02B01-02, SW58 KS-2P02B01-02, SW59 KS-2P02B01-02, SW6 KS-2P02B01-02, SW60 RESET, SW61 BOOTSEL (VERIFY), SW62 PWR MSK-12C02, SW7 KS-2P02B01-02, SW8 KS-2P02B01-02, SW9 KS-2P02B01-02, U1 RP2040, U2 MCP73831-2ACI/OT, U3 AP2112K-3.3, U4 USBLC6-2SC6, U5 W25Q16JVUXIQ, U6 CYW43439, U7 SN74AHCT1G125DBVR, Y1 12MHz, Y2 37.4MHz

Commit message: sent to PCBWay
Parts:
- removed ANT1: 2450AT18B100E, kbd:ANT_JOHANSON_2450AT18B100, symbol kbd:ANT_JOHANSON
- removed C17: 1.2p (ref: Johanson), kbd:RC_0402, symbol kbd:C_kbd
- removed C18: DNP (VERIFY, tune), kbd:RC_0402, symbol kbd:C_kbd
- removed C20, C24: 4.7u, kbd:RC_0603, symbol kbd:C_kbd
- removed C21, C27, C28, C29: 100n (VERIFY), kbd:RC_0603, symbol kbd:C_kbd
- removed C22: 2.2u, kbd:RC_0603, symbol kbd:C_kbd
- removed C23: 2.2u (VERIFY), kbd:RC_0603, symbol kbd:C_kbd
- removed C25, C26: 1u, kbd:RC_0603, symbol kbd:C_kbd
- removed C30, C31: 27p, kbd:RC_0603, symbol kbd:C_kbd
- removed L2: 2.7nH (ref: Johanson), kbd:RC_0201, symbol kbd:R_kbd
- removed L3: 2.2uH, kbd:RC_0603, symbol kbd:R_kbd
- removed R12: 22, kbd:RC_0603, symbol kbd:R_kbd
- removed R13: 0 (ref: Pico W), kbd:RC_0603, symbol kbd:R_kbd
- removed U6: CYW43439, kbd:CYW43439_WLBGA63, symbol kbd:CYW43439_WLBGA63
- removed Y2: 37.4MHz, kbd:XTAL_3225, symbol kbd:XTAL
- added R14: 470, kbd:RC_0603, symbol kbd:R_kbd
- added R15: 10k, kbd:RC_0603, symbol kbd:R_kbd
- added U6: RM2, kbd:RM2_RMC20452T, symbol kbd:RM2
- D1, D10, D11, D12, D13, D14, D15, D16, D17, D18, D19, D2, D20, D21, D22, D23, D24, D25, D26, D27, D28, D29, D3, D30, D31, D32, D33, D34, D35, D36, D37, D38, D39, D4, D40, D41, D42, D43, D44, D45, D46, D47, D48, D49, D5, D50, D51, D52, D53, D54, D55, D56, D57, D58, D59, D6, D7, D8, D9: BOM Comments (none) -> SOD-123; MPN (none) -> 1N4148W-E3-08; Manufacturer (none) -> Vishay
- D60: BOM Comments (none) -> Schottky 1A 40V SOD-123; MPN (none) -> B5819W; Manufacturer (none) -> MDD
- J1: BOM Comments (none) -> USB-C 16P; MPN (none) -> TYPE-C-31-M-12; Manufacturer (none) -> Korean Hroparts
- J2: BOM Comments (none) -> battery, back side; MPN (none) -> SM02B-SRSS-TB(LF)(SN); Manufacturer (none) -> JST
- Q1: MPN (none) -> DMG3415U-7; Manufacturer (none) -> Diodes Incorporated
- RGB1, RGB10, RGB11, RGB12, RGB13, RGB14, RGB15, RGB16, RGB17, RGB18, RGB19, RGB2, RGB20, RGB21, RGB22, RGB23, RGB24, RGB25, RGB26, RGB27, RGB28, RGB29, RGB3, RGB30, RGB31, RGB32, RGB33, RGB34, RGB35, RGB36, RGB37, RGB38, RGB39, RGB4, RGB40, RGB41, RGB42, RGB43, RGB44, RGB45, RGB46, RGB47, RGB48, RGB49, RGB5, RGB50, RGB51, RGB52, RGB53, RGB54, RGB55, RGB56, RGB57, RGB58, RGB59, RGB6, RGB7, RGB8, RGB9: BOM Comments (none) -> reverse-mount RGB; MPN (none) -> SK6812MINI-E; Manufacturer (none) -> OPSCO
- SW60: BOM Comments (none) -> 6x6 THT tactile switch, hand-solder
- SW61: value BOOTSEL (VERIFY) -> BOOTSEL; BOM Comments (none) -> 6x6 THT tactile switch, hand-solder
- SW62: BOM Comments (none) -> slide switch; MPN (none) -> MSK-12C02; Manufacturer (none) -> Shou Han
- U1: MPN (none) -> SC0914; Manufacturer (none) -> Raspberry Pi
- U2: MPN (none) -> MCP73831T-2ACI/OT; Manufacturer (none) -> Microchip
- U3: MPN (none) -> AP2112K-3.3TRG1; Manufacturer (none) -> Diodes Incorporated
- U4: MPN (none) -> USBLC6-2SC6; Manufacturer (none) -> STMicroelectronics
- U5: MPN (none) -> W25Q16JVUXIQ TR; Manufacturer (none) -> Winbond
- U7: MPN (none) -> SN74AHCT1G125DBVR; Manufacturer (none) -> Texas Instruments
- Y1: BOM Comments (none) -> 12MHz 3225 CL=10pF (RPi-recommended); MPN (none) -> ABM8-272-T3; Manufacturer (none) -> Abracon
Connections:
- net QSPI_SD1: now also U1.54 (QSPI_SD1); no longer U1.55 (QSPI_SD1)
- net QSPI_SD2: now also U1.55 (QSPI_SD2); no longer U1.54 (QSPI_SD2)
- net WL_DATA: now reaches U1.36 (GPIO24)
- net WL_DATA: now also R14.2, R15.2
- net WL_CS: now reaches U1.37 (GPIO25)
- net WL_CLK: now reaches U1.41 (GPIO29/ADC3)
- net BT_DEV_WAKE: no longer names the net of U1.30 (GPIO19)
- net BT_HOST_WAKE: no longer names the net of U1.40 (GPIO28/ADC2)
- net BT_REG_ON: no longer names the net of U1.29 (GPIO18)
- net BT_UART_CTS_N renamed WL_ON
- net BT_UART_RTS_N: no longer names the net of U1.34 (GPIO22/UART1_CTS)
- net BT_UART_RXD: no longer names the net of U1.31 (GPIO20/UART1_TX)
- net BT_UART_TXD: no longer names the net of U1.32 (GPIO21/UART1_RX)
- new net WL_DOUT: R14.1
- new net WL_IRQ: R15.1
- no-connect marks 9 -> 18
Other:
- note added: "Charging works with power switch OFF (charger connects before switch). BOOTSEL+RESET = USB mass-storage bootloader mode."
- note removed: "Charging works with power switch OFF (charger connects before switch). BOOTSEL+RESET = USB mass-storage bootloader mode (VERIFY)."
